Commit message: update the urdf file

File: src/dual_arm_description/urdf/left_arm.xacro (robot description, xacro)
@@ -1,11 +1,10 @@
 <?xml version="1.0"?>
 <robot xmlns:xacro="http://www.ros.org/wiki/xacro">
-  <xacro:macro name="default_inertial">
+  <link name="left_base">
     <inertial>
-      <mass value="0.1"/>
-      <inertia ixx="1e-4" ixy="0" ixz="0" iyy="1e-4" iyz="0" izz="1e-4"/>
+      <origin xyz="0.00032267 4.798E-05 0.04066353" rpy="0 0 0"/>
+      <mass value="1.1962"/>
+      <inertia ixx="0.00107329" ixy="-1.68E-06" ixz="-1.05E-05" iyy="0.00107003" iyz="-3.43E-06" izz="0.00127315"/>
     </inertial>
-  </xacro:macro>
-  <link name="left_base">
     <visual>
       <geometry>
@@ -19,13 +18,11 @@
       </geometry>
     </collision>
-    <xacro:default_inertial/>
   </link>
-  <!-- <joint name="world_to_left_base" type="fixed">
-    <origin xyz="-0.1 0 1.0" rpy="0 -1.57079632679 0"/>
-    <parent link="world"/>
-    <child link="left_base"/>
-  </joint> -->
-  <!-- left Arm Links -->
   <link name="left_link1">
+    <inertial>
+      <origin xyz="0.00002347 0.00557150 -0.03075998" rpy="0 0 0"/>
+      <mass value="1.9705"/>
+      <inertia ixx="0.00492293" ixy="0.00000550" ixz="0.00000193" iyy="0.00526513" iyz="0.00033232" izz="0.00188107"/>
+    </inertial>
     <visual>
       <origin xyz="0.0000008 0 0"/>
@@ -41,5 +38,4 @@
       </geometry>
     </collision>
-    <xacro:default_inertial/>
   </link>
   <joint name="left_joint1" type="revolute">
@@ -47,7 +43,12 @@
     <child link="left_link1"/>
     <axis xyz="0 0 1"/>
-    <limit lower="-3.05433" upper="3.05433" effort="100" velocity="6.28"/>
+    <limit lower="-3.1067" upper="3.1067" effort="108" velocity="3.1416"/>
   </joint>
   <link name="left_link2">
+    <inertial>
+      <origin xyz="0.00013483 0.06170460 0.00950639" rpy="0 0 0"/>
+      <mass value="2.24398"/>
+      <inertia ixx="0.01194933" ixy="0.00000336" ixz="0.00000091" iyy="0.00361581" iyz="-0.00132804" izz="0.01098356"/>
+    </inertial>
     <visual>
       <geometry><mesh filename="package://dual_arm_description/meshes/link2_Mesh.obj"/></geometry>
@@ -57,5 +58,4 @@
       <geometry><mesh filename="package://dual_arm_description/meshes/link2_Mesh.obj"/></geometry>
     </collision>
-    <xacro:default_inertial/>
   </link>
   <joint name="left_joint2" type="revolute">
@@ -64,7 +64,12 @@
     <origin xyz="0 0 0.1743"/>
     <axis xyz="0 -1 0"/>
-    <limit lower="-2.00713" upper="2.00713" effort="100" velocity="6.28"/>
+    <limit lower="-2.0944" upper="2.0944" effort="108" velocity="3.1416"/>
   </joint>
   <link name="left_link3">
+    <inertial>
+      <origin xyz="0.00968562 0.00246599 -0.04627302" rpy="0 0 0"/>
+      <mass value="1.9242"/>
+      <inertia ixx="0.00718224" ixy="0.00004413" ixz="0.00089552" iyy="0.00762563" iyz="0.00022096" izz="0.00178597"/>
+    </inertial>
     <visual>
       <origin rpy="0 0 3.1415"/>
@@ -85,5 +90,4 @@
       <geometry><mesh filename="package://dual_arm_description/meshes/LINK3_UPPER_Mesh.obj"/></geometry>
     </collision>
-    <xacro:default_inertial/>
   </link>
   <joint name="left_joint3" type="revolute">
@@ -91,7 +95,12 @@
     <child link="left_link3"/>
     <axis xyz="0 0 1"/>
-    <limit lower="-3.05433" upper="3.05433" effort="100" velocity="6.28"/>
+    <limit lower="-3.1067" upper="3.1067" effort="66" velocity="3.1416"/>
   </joint>
   <link name="left_link4">
+    <inertial>
+      <origin xyz="0.00850411 -0.04718223 0.00941509" rpy="0 0 0"/>
+      <mass value="1.6085"/>
+      <inertia ixx="0.00580480" ixy="-0.00066669" ixz="-0.00012722" iyy="0.00223807" iyz="0.00070523" izz="0.00533060"/>
+    </inertial>
     <visual>
       <origin rpy="0 0 -3.1415"/>
@@ -103,5 +112,4 @@
       <geometry><mesh filename="package://dual_arm_description/meshes/LINK4_Mesh.obj"/></geometry>
     </collision>
-    <xacro:default_inertial/>
   </link>
   <joint name="left_joint4" type="revolute">
@@ -110,7 +118,12 @@
     <origin xyz="-0.018 0 0.287"/>
     <axis xyz="0 -1 0"/>
-    <limit lower="-2.44346" upper="0.959931" effort="100" velocity="6.28"/>
+    <limit lower="-2.5307" upper="1.0472" effort="66" velocity="3.1416"/>
   </joint>
   <link name="left_link5">
+    <inertial>
+      <origin xyz="0.00051127 0.00101064 -0.11271739" rpy="0 0 0"/>
+      <mass value="2.0883"/>
+      <inertia ixx="0.00626603" ixy="0.00004009" ixz="0.00005338" iyy="0.00564387" iyz="-0.00006193" izz="0.00243632"/>
+    </inertial>
     <visual>
       <geometry><mesh filename="package://dual_arm_description/meshes/LINK5_Mesh.obj"/></geometry>
@@ -120,5 +133,4 @@
       <geometry><mesh filename="package://dual_arm_description/meshes/LINK5_Mesh.obj"/></geometry>
     </collision>
-    <xacro:default_inertial/>
   </link>
   <joint name="left_joint5" type="revolute">
@@ -127,7 +139,12 @@
     <origin xyz="0.018 0 0.314"/>
     <axis xyz="0 0 1"/>
-    <limit lower="-3.05433" upper="3.05433" effort="100" velocity="6.28"/>
+    <limit lower="-3.1067" upper="3.1067" effort="18" velocity="3.1416"/>
   </joint>
   <link name="left_link6">
+    <inertial>
+      <origin xyz="0.00032659 0.00531336 -0.00030182" rpy="0 0 0"/>
+      <mass value="0.72496"/>
+      <inertia ixx="0.00046040" ixy="0.00000189" ixz="0.00000083" iyy="0.00051716" iyz="-0.00000346" izz="0.00042521"/>
+    </inertial>
     <visual>
       <geometry><mesh filename="package://dual_arm_description/meshes/LINK6_Mesh.obj"/></geometry>
@@ -137,5 +154,4 @@
       <geometry><mesh filename="package://dual_arm_description/meshes/LINK6_Mesh.obj"/></geometry>
     </collision>
-    <xacro:default_inertial/>
   </link>
   <joint name="left_joint6" type="revolute">
@@ -143,12 +159,16 @@
     <child link="left_link6"/>
     <axis xyz="0 -1 0"/>
-    <limit lower="-0.959931" upper="0.959931" effort="100" velocity="6.28"/>
+    <limit lower="-1.0472" upper="1.0472" effort="18" velocity="3.1416"/>
   </joint>
   <link name="left_ttt">
+    <inertial>
+      <origin xyz="-0.00009108 -0.03153255 0.00889371" rpy="0 0 0"/>
+      <mass value="0.68606"/>
+      <inertia ixx="0.00173687" ixy="-0.00000345" ixz="-0.00000116" iyy="0.00089035" iyz="0.00030680" izz="0.00139406"/>
+    </inertial>
     <visual>
       <origin rpy="3.1415 -1.5707 0"/>
       <geometry><mesh filename="package://dual_arm_description/meshes/tn__T_Arm_MarvinM6SLCCS_WKe8HJ_01_Mesh.obj"/></geometry>
     </visual>
-    <xacro:default_inertial/>
   </link>
   <joint name="left_joint7" type="revolute">
@@ -156,5 +176,5 @@
     <child link="left_ttt"/>
     <axis xyz="1 0 0"/>
-    <limit lower="-1.48353" upper="1.48353" effort="100" velocity="6.28"/>
+    <limit lower="-1.5708" upper="1.5708" effort="18" velocity="3.1416"/>
   </joint>
   <link name="left_flange"/>
@@ -162,5 +182,5 @@
     <parent link="left_ttt"/>
     <child link="left_flange"/>
-    <origin xyz="0 0 0.088"/>
+    <origin xyz="0 0 0.088" rpy="0 0 0"/>
   </joint>
 </robot>

File: src/dual_arm_description/urdf/right_arm.xacro (robot description, xacro)
@@ -1,11 +1,10 @@
 <?xml version="1.0"?>
 <robot xmlns:xacro="http://www.ros.org/wiki/xacro">
-  <xacro:macro name="default_inertial">
+  <link name="right_base">
     <inertial>
-      <mass value="0.1"/>
-      <inertia ixx="1e-4" ixy="0" ixz="0" iyy="1e-4" iyz="0" izz="1e-4"/>
+      <origin xyz="0.00032267 4.798E-05 0.04066353" rpy="0 0 0"/>
+      <mass value="1.1962"/>
+      <inertia ixx="0.00107329" ixy="-1.68E-06" ixz="-1.05E-05" iyy="0.00107003" iyz="-3.43E-06" izz="0.00127315"/>
     </inertial>
-  </xacro:macro>
-  <link name="right_base">
     <visual>
       <geometry>
@@ -19,13 +18,11 @@
       </geometry>
     </collision>
-    <xacro:default_inertial/>
   </link>
-  <!-- <joint name="world_to_right_base" type="fixed">
-    <origin xyz="0.1 0 1.0" rpy="0 1.57079632679 0"/>
-    <parent link="world"/>
-    <child link="right_base"/>
-  </joint> -->
-  <!-- Right Arm Links -->
   <link name="right_link1">
+    <inertial>
+      <origin xyz="0.00002347 0.00557150 -0.03075998" rpy="0 0 0"/>
+      <mass value="1.9705"/>
+      <inertia ixx="0.00492293" ixy="0.00000550" ixz="0.00000193" iyy="0.00526513" iyz="0.00033232" izz="0.00188107"/>
+    </inertial>
     <visual>
       <origin xyz="0.0000008 0 0"/>
@@ -41,5 +38,4 @@
       </geometry>
     </collision>
-    <xacro:default_inertial/>
   </link>
   <joint name="right_joint1" type="revolute">
@@ -47,7 +43,12 @@
     <child link="right_link1"/>
     <axis xyz="0 0 1"/>
-    <limit lower="-3.05433" upper="3.05433" effort="100" velocity="6.28"/>
+    <limit lower="-3.1067" upper="3.1067" effort="108" velocity="3.1416"/>
   </joint>
   <link name="right_link2">
+    <inertial>
+      <origin xyz="0.00013483 0.06170460 0.00950639" rpy="0 0 0"/>
+      <mass value="2.24398"/>
+      <inertia ixx="0.01194933" ixy="0.00000336" ixz="0.00000091" iyy="0.00361581" iyz="-0.00132804" izz="0.01098356"/>
+    </inertial>
     <visual>
       <geometry><mesh filename="package://dual_arm_description/meshes/link2_Mesh.obj"/></geometry>
@@ -57,5 +58,4 @@
       <geometry><mesh filename="package://dual_arm_description/meshes/link2_Mesh.obj"/></geometry>
     </collision>
-    <xacro:default_inertial/>
   </link>
   <joint name="right_joint2" type="revolute">
@@ -64,7 +64,12 @@
     <origin xyz="0 0 0.1743"/>
     <axis xyz="0 1 0"/>
-    <limit lower="-2.00713" upper="2.00713" effort="100" velocity="6.28"/>
+    <limit lower="-2.0944" upper="2.0944" effort="108" velocity="3.1416"/>
   </joint>
   <link name="right_link3">
+    <inertial>
+      <origin xyz="0.00968562 0.00246599 -0.04627302" rpy="0 0 0"/>
+      <mass value="1.9242"/>
+      <inertia ixx="0.00718224" ixy="0.00004413" ixz="0.00089552" iyy="0.00762563" iyz="0.00022096" izz="0.00178597"/>
+    </inertial>
     <visual>
       <origin rpy="0 0 3.1415"/>
@@ -85,5 +90,4 @@
       <geometry><mesh filename="package://dual_arm_description/meshes/LINK3_UPPER_Mesh.obj"/></geometry>
     </collision>
-    <xacro:default_inertial/>
   </link>
   <joint name="right_joint3" type="revolute">
@@ -91,7 +95,12 @@
     <child link="right_link3"/>
     <axis xyz="0 0 1"/>
-    <limit lower="-3.05433" upper="3.05433" effort="100" velocity="6.28"/>
+    <limit lower="-3.1067" upper="3.1067" effort="66" velocity="3.1416"/>
   </joint>
   <link name="right_link4">
+    <inertial>
+      <origin xyz="0.00850411 -0.04718223 0.00941509" rpy="0 0 0"/>
+      <mass value="1.6085"/>
+      <inertia ixx="0.00580480" ixy="-0.00066669" ixz="-0.00012722" iyy="0.00223807" iyz="0.00070523" izz="0.00533060"/>
+    </inertial>
     <visual>
       <origin rpy="0 0 -3.1415"/>
@@ -103,5 +112,4 @@
       <geometry><mesh filename="package://dual_arm_description/meshes/LINK4_Mesh.obj"/></geometry>
     </collision>
-    <xacro:default_inertial/>
   </link>
   <joint name="right_joint4" type="revolute">
@@ -110,7 +118,12 @@
     <origin xyz="-0.018 0 0.287"/>
     <axis xyz="0 1 0"/>
-    <limit lower="-2.44346" upper="0.959931" effort="100" velocity="6.28"/>
+    <limit lower="-2.5307" upper="1.0472" effort="66" velocity="3.1416"/>
   </joint>
   <link name="right_link5">
+    <inertial>
+      <origin xyz="-0.00051127 -0.00101064 -0.11271739" rpy="0 0 0"/>
+      <mass value="2.0883"/>
+      <inertia ixx="0.00626603" ixy="0.00004009" ixz="-0.00005338" iyy="0.00564387" iyz="0.00006193" izz="0.00243632"/>
+    </inertial>
     <visual>
       <geometry><mesh filename="package://dual_arm_description/meshes/LINK5_Mesh.obj"/></geometry>
@@ -120,5 +133,4 @@
       <geometry><mesh filename="package://dual_arm_description/meshes/LINK5_Mesh.obj"/></geometry>
     </collision>
-    <xacro:default_inertial/>
   </link>
   <joint name="right_joint5" type="revolute">
@@ -127,7 +139,12 @@
     <origin xyz="0.018 0 0.314"/>
     <axis xyz="0 0 1"/>
-    <limit lower="-3.05433" upper="3.05433" effort="100" velocity="6.28"/>
+    <limit lower="-3.1067" upper="3.1067" effort="18" velocity="3.1416"/>
   </joint>
   <link name="right_link6">
+    <inertial>
+      <origin xyz="0.00032659 -0.00531336 0.00030182" rpy="0 0 0"/>
+      <mass value="0.72496"/>
+      <inertia ixx="0.00046040" ixy="-0.00000189" ixz="-0.00000083" iyy="0.00051716" iyz="-0.00000346" izz="0.00042521"/>
+    </inertial>
     <visual>
       <geometry><mesh filename="package://dual_arm_description/meshes/LINK6_Mesh.obj"/></geometry>
@@ -137,5 +154,4 @@
       <geometry><mesh filename="package://dual_arm_description/meshes/LINK6_Mesh.obj"/></geometry>
     </collision>
-    <xacro:default_inertial/>
   </link>
   <joint name="right_joint6" type="revolute">
@@ -143,12 +159,16 @@
     <child link="right_link6"/>
     <axis xyz="0 1 0"/>
-    <limit lower="-0.959931" upper="0.959931" effort="100" velocity="6.28"/>
+    <limit lower="-1.0472" upper="1.0472" effort="18" velocity="3.1416"/>
   </joint>
   <link name="right_ttt">
+    <inertial>
+      <origin xyz="-0.00009108 -0.03153255 0.00889371" rpy="0 0 0"/>
+      <mass value="0.68606"/>
+      <inertia ixx="0.00173687" ixy="-0.00000345" ixz="-0.00000116" iyy="0.00089035" iyz="0.00030680" izz="0.00139406"/>
+    </inertial>
     <visual>
       <origin rpy="3.1415 -1.5707 0"/>
       <geometry><mesh filename="package://dual_arm_description/meshes/tn__T_Arm_MarvinM6SLCCS_WKe8HJ_01_Mesh.obj"/></geometry>
     </visual>
-    <xacro:default_inertial/>
   </link>
   <joint name="right_joint7" type="revolute">
@@ -156,5 +176,5 @@
     <child link="right_ttt"/>
     <axis xyz="1 0 0"/>
-    <limit lower="-1.48353" upper="1.48353" effort="100" velocity="6.28"/>
+    <limit lower="-1.5708" upper="1.5708" effort="18" velocity="3.1416"/>
   </joint>
   <link name="right_flange"/>
@@ -162,5 +182,5 @@
     <parent link="right_ttt"/>
     <child link="right_flange"/>
-    <origin xyz="0 0 0.088"/>
+    <origin xyz="0 0 0.088" rpy="0 0 0"/>
   </joint>
 </robot>
